File: hardware/stow-minipcie-single.kicad_pcb (KiCad board)
At the start: 2 copper layers, 30 x 51 mm, 10 parts, among them P1 mPCIe, P2 USB, U1 SM200, U2 FT232RL

Commit message: Add back silkscreen.
Parts:
- added G***: LOGO, _CrumpSymbols:Symbol_OSHW-Logo_12.5mm_NoText_Silkscreen, B.Cu at (86.5, 67.5)
Other:
- board text added: "(S)ynapse (T)actical (O)ccluded (W)ireless"
- board text added: "@tylercrumpton"
- board text added: "CC-BY-SA 4.0"
- board text added: "Module"
- board text added: "S.T.O.W."
- board text added: "v0.0"
Changed lines of the file:
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@@
     (area 71.549999 55.999999 101.650001 107.050001)
     (thickness 1.6)
-    (drawings 20)
+    (drawings 26)
     (tracks 484)
     (zones 0)
-    (modules 10)
+    (modules 11)
     (nets 79)
   )
@@
     (mod_text_size 1 1)
     (mod_text_width 0.15)
-    (pad_size 0.6 2)
+    (pad_size 5.8 5.8)
     (pad_drill 0)
     (pad_to_mask_clearance 0)
@@
     (pad 52 smd rect (at 11.9 -1.55) (size 0.6 2) (layers B.Cu B.Paste B.Mask)
       (net 6 VCC))
-    (pad "" connect rect (at 12.1 -23.9) (size 5.8 5.8) (layers B.SilkS))
+    (pad "" connect rect (at 12.1 -23.9) (size 5.8 5.8) (layers Dwgs.User))
     (pad "" np_thru_hole circle (at -12.1 -48.05) (size 2.6 2.6) (drill 2.6) (layers *.Cu *.Mask F.SilkS))
-    (pad "" connect rect (at 12.1 -9) (size 5.8 5.8) (layers B.SilkS))
-    (pad "" connect rect (at -12.1 -9) (size 5.8 5.8) (layers B.SilkS))
-    (pad "" connect rect (at -12.1 -23.9) (size 5.8 5.8) (layers B.SilkS))
+    (pad "" connect rect (at 12.1 -9) (size 5.8 5.8) (layers Dwgs.User))
+    (pad "" connect rect (at -12.1 -9) (size 5.8 5.8) (layers Dwgs.User))
+    (pad "" connect rect (at -12.1 -23.9) (size 5.8 5.8) (layers Dwgs.User))
     (pad "" np_thru_hole circle (at 12.1 -48.05) (size 2.6 2.6) (drill 2.6) (layers *.Cu *.Mask F.SilkS))
     (pad "" connect rect (at -12.1 -48.05) (size 5.8 5.8) (layers B.SilkS))
     (pad "" connect rect (at 12.1 -48.05) (size 5.8 5.8) (layers B.SilkS))
-    (pad "" connect rect (at -12.1 -33.35) (size 5.8 5.8) (layers B.SilkS))
-    (pad "" connect rect (at 12.1 -33.35) (size 5.8 5.8) (layers B.SilkS))
+    (pad "" connect rect (at -12.1 -33.35) (size 5.8 5.8) (layers Dwgs.User))
+    (pad "" connect rect (at 12.1 -33.35) (size 5.8 5.8) (layers Dwgs.User))
+  )
+  (module _CrumpSymbols:Symbol_OSHW-Logo_12.5mm_NoText_Silkscreen (layer B.Cu)
+    (at 86.5 67.5 180)
+    (fp_text reference G*** (at 0 0 180) (layer B.SilkS) hide
+      (effects (font (thickness 0.3)) (justify mirror))
+    )
+    (fp_text value LOGO (at 0.75 0 180) (layer B.SilkS) hide
+      (effects (font (thickness 0.3)) (justify mirror))
+    )
+    (fp_poly (pts (xy 6.186444 -1.510795) (xy 5.739055 -1.598946) (xy 5.407619 -1.66271) (xy 5.083407 -1.72269)
+      (xy 4.964541 -1.743777) (xy 4.770372 -1.792122) (xy 4.639717 -1.882689) (xy 4.527433 -2.059029)
+      (xy 4.437704 -2.252043) (xy 4.282738 -2.614376) (xy 4.201874 -2.87563) (xy 4.199782 -3.089168)
+      (xy 4.281135 -3.308355) (xy 4.450602 -3.586557) (xy 4.570131 -3.764897) (xy 5.006375 -4.411382)
+      (xy 4.416979 -5.016138) (xy 3.827584 -5.620893) (xy 3.152085 -5.177415) (xy 2.476586 -4.733937)
+      (xy 2.170689 -4.879809) (xy 1.96805 -4.961694) (xy 1.837057 -4.987377) (xy 1.820353 -4.981242)
+      (xy 1.774541 -4.891911) (xy 1.675942 -4.672863) (xy 1.536255 -4.350958) (xy 1.367177 -3.953053)
+      (xy 1.232971 -3.632568) (xy 0.690029 -2.328333) (xy 1.066889 -2.002357) (xy 1.408976 -1.657933)
+      (xy 1.614569 -1.315009) (xy 1.708301 -0.923012) (xy 1.721118 -0.659281) (xy 1.644396 -0.14112)
+      (xy 1.427912 0.30732) (xy 1.093668 0.663905) (xy 0.663664 0.906504) (xy 0.159904 1.012983)
+      (xy 0.055747 1.016) (xy -0.470501 0.94035) (xy -0.919998 0.728237) (xy -1.275002 0.401916)
+      (xy -1.517769 -0.016356) (xy -1.630559 -0.504323) (xy -1.595628 -1.039729) (xy -1.593 -1.052173)
+      (xy -1.512786 -1.321452) (xy -1.379524 -1.554837) (xy -1.157097 -1.810103) (xy -1.056396 -1.910529)
+      (xy -0.610517 -2.345846) (xy -1.151871 -3.642313) (xy -1.334817 -4.07696) (xy -1.496677 -4.454953)
+      (xy -1.625708 -4.749392) (xy -1.710173 -4.933377) (xy -1.736676 -4.982231) (xy -1.832647 -4.97664)
+      (xy -2.019586 -4.90985) (xy -2.090349 -4.877747) (xy -2.40057 -4.729813) (xy -3.029339 -5.158906)
+      (xy -3.314754 -5.34926) (xy -3.547541 -5.496287) (xy -3.692612 -5.578192) (xy -3.720164 -5.588)
+      (xy -3.801954 -5.530818) (xy -3.971288 -5.37706) (xy -4.199599 -5.153405) (xy -4.351232 -4.998605)
+      (xy -4.920244 -4.409211) (xy -4.492122 -3.774762) (xy -4.301465 -3.479634) (xy -4.154501 -3.228182)
+      (xy -4.073255 -3.059195) (xy -4.064 -3.02078) (xy -4.095988 -2.876332) (xy -4.176874 -2.636217)
+      (xy -4.284047 -2.358261) (xy -4.394891 -2.100289) (xy -4.486795 -1.920128) (xy -4.505155 -1.89269)
+      (xy -4.631335 -1.815355) (xy -4.848115 -1.749891) (xy -4.892517 -1.741406) (xy -5.167395 -1.691793)
+      (xy -5.503115 -1.628387) (xy -5.65439 -1.598946) (xy -6.101779 -1.510795) (xy -6.077723 -0.649564)
+      (xy -6.053667 0.211667) (xy -5.296156 0.359578) (xy -4.955127 0.431557) (xy -4.679353 0.499833)
+      (xy -4.509854 0.553789) (xy -4.478509 0.571245) (xy -4.41746 0.677085) (xy -4.315322 0.893142)
+      (xy -4.194741 1.171385) (xy -3.97111 1.70777) (xy -4.441899 2.395909) (xy -4.912688 3.084048)
+      (xy -4.342448 3.658691) (xy -4.086931 3.906926) (xy -3.869443 4.101234) (xy -3.720839 4.214885)
+      (xy -3.67918 4.233334) (xy -3.57147 4.187923) (xy -3.363347 4.066639) (xy -3.09228 3.891899)
+      (xy -2.971637 3.81) (xy -2.687838 3.620163) (xy -2.454218 3.474369) (xy -2.307181 3.394903)
+      (xy -2.280118 3.386667) (xy -2.167354 3.416216) (xy -1.946304 3.493622) (xy -1.669454 3.600306)
+      (xy -1.135793 3.813946) (xy -0.970064 4.637473) (xy -0.804334 5.461) (xy 0.022092 5.485244)
+      (xy 0.396071 5.496272) (xy 0.652567 5.485958) (xy 0.819385 5.428102) (xy 0.92433 5.296505)
+      (xy 0.995208 5.064969) (xy 1.059825 4.707294) (xy 1.098855 4.470685) (xy 1.207741 3.819037)
+      (xy 1.747761 3.602852) (xy 2.031832 3.493904) (xy 2.25712 3.416228) (xy 2.374697 3.386667)
+      (xy 2.479332 3.432585) (xy 2.683861 3.55513) (xy 2.951114 3.73149) (xy 3.064418 3.810001)
+      (xy 3.34719 4.001347) (xy 3.583047 4.147671) (xy 3.734283 4.226094) (xy 3.762048 4.233334)
+      (xy 3.859384 4.176585) (xy 4.042694 4.024195) (xy 4.280969 3.802947) (xy 4.425555 3.660261)
+      (xy 4.994236 3.087189) (xy 4.527888 2.390632) (xy 4.06154 1.694075) (xy 4.282289 1.164538)
+      (xy 4.402631 0.887059) (xy 4.503976 0.673276) (xy 4.563175 0.571245) (xy 4.668247 0.52774)
+      (xy 4.898961 0.4649) (xy 5.214296 0.393346) (xy 5.380822 0.359578) (xy 6.138333 0.211667)
+      (xy 6.162389 -0.649564) (xy 6.186444 -1.510795) (xy 6.186444 -1.510795)) (layer B.SilkS) (width 0.1))
+  )
+  (gr_text v0.0 (at 76.75 99.75) (layer B.SilkS)
+    (effects (font (size 1.5 1.5) (thickness 0.3)) (justify mirror))
+  )
+  (gr_text Module (at 86.5 88.5) (layer B.SilkS)
+    (effects (font (size 2 3) (thickness 0.5)) (justify mirror))
+  )
+  (gr_text "(S)ynapse\n(T)actical\n(O)ccluded\n(W)ireless\n" (at 98.25 96) (layer B.SilkS)
+    (effects (font (size 1.5 1.5) (thickness 0.3) italic) (justify left mirror))
+  )
+  (gr_text S.T.O.W. (at 86.5 84.5) (layer B.SilkS)
+    (effects (font (size 4 4) (thickness 1)) (justify mirror))
+  )
+  (gr_text @tylercrumpton (at 86.5 76.5) (layer B.SilkS)
+    (effects (font (size 1.5 1.5) (thickness 0.3)) (justify mirror))
+  )
+  (gr_text "CC-BY-SA 4.0" (at 86.5 74.5) (layer B.SilkS)
+    (effects (font (size 1.5 1.5) (thickness 0.3)) (justify mirror))
   )
   (gr_text D+ (at 91.75 62.5) (layer F.SilkS)
