File: hardware/stow-minipcie-single.kicad_pcb (KiCad board)
At the start: 2 copper layers, 30 x 51 mm, 11 parts, among them P1 mPCIe, P2 USB, U1 SM200, U2 FT232RL

Commit message: Change version label to v1.0.
Other:
- board text added: "v1.0"
- board text removed: "v0.0"
